File: KiCAD/UPDI Board.kicad_sch (KiCad schematic)
At the start: 18 parts, among them J1 AVR UPDI Header, J10 Primary Header, J12 Second Header, J13 RS485, J14 UART0, J15 UPDI, J16 Voltage in, J17 UART1, U7 MAX3072E

Commit message: .
Parts:
- added C19: 220n, Capacitor_SMD:C_0805_2012Metric_Pad1.18x1.45mm_HandSolder, symbol Device:C_Small
- added R18, R19: 10, Resistor_SMD:R_0805_2012Metric_Pad1.20x1.40mm_HandSolder, symbol Device:R_Small
- C18: value 100nF -> 100n
Connections:
- net +5V: now also C19.1
- net A: now also R18.2; no longer J13.2 (Pin_2), R17.2
- net B: now also R19.2; no longer J13.3 (Pin_3), R17.1
- net GND: now also C19.2
- new net: J13.2 (Pin_2), R17.2, R18.1
- new net: J13.3 (Pin_3), R17.1, R19.1
Other:
- moved on the sheet: R17

Commit message: .
Other:
- note removed: "https://github.com/MCUdude/microUPDI"
