File: KiCAD/UPDI Board.kicad_sch (KiCad schematic)
At the start: 21 parts, among them J1 AVR UPDI Header, J10 Primary Header, J12 Second Header, J13 RS485, J14 UART0, J15 UPDI, J16 Voltage in, J17 UART1, U7 MAX3072E

Commit message: Clean up and add LED
Parts:
- added D13: Feedback LED, LED_SMD:LED_0805_2012Metric_Pad1.15x1.40mm_HandSolder, symbol Device:LED_Small_Filled
- added R20: 470, Resistor_SMD:R_0805_2012Metric_Pad1.20x1.40mm_HandSolder, symbol Device:R_Small
Connections:
- net GND: now also R20.2
- net at J1.3 (Pin_3): now also D13.2 (A)
- new net: D13.1 (K), R20.1
- no-connect marks 4 -> 3
Other:
- note added: "Poka Yoke footprint can be removed when confirmed pins are the right way round"
- note added: "RS485 is only guarenteed for 5 VDC, TBC"
- note added: "The Feedback LED is not part of the AVR HDPI header standard, however, I have included it on the un-used pin so that I can have a status/feedback LED for visual feedback from the microcontroller."
- note removed: "RS485 is only guarenteed for 5V"
- moved on the sheet: C19, D11, J1, J10, J12, J13, J14, J15, J17, R1, R14, R15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
